File: c64-umd/c64-umd.kicad_pcb (KiCad board)
At the start: 2 copper layers, 20.3 x 83.8 mm, 11 parts, among them CON101 C64-CONN, CON102 UMD-CONN, Q101 SMMBT3904LT1G, U101 MC74HC589ADTR2G

Commit message: prelim routing complete, review before 0.1 release
Parts:
- removed the G*** at (148.1, 71.4)
- moved R103 7.77 mm to (147.3, 145.3), turned to 0 degrees
- moved R101 3.73 mm to (150.7, 77.2)
- moved D101 1.84 mm to (150.7, 144.1), turned to 180 degrees
- moved Q101 1.46 mm to (153.3, 77.0)
- moved C101 0.51 mm to (154.4, 68.5)
Connections:
- CON102 pad 10: +5V -> (no net)
- CON102 pad 4: /~ROMH -> /~EXROM
- CON102 pad 5: /~EXROM -> /~GAME
- CON102 pad 55: GND -> (no net)
- CON102 pad 6: /~GAME -> /Phi2
- CON102 pad 60: /Phi2 -> /~IO2
- CON102 pad 61: /~IO2 -> /~ROML
- CON102 pad 7: /~IO1 -> /~ROMH
- CON102 pad 8: /~ROML -> /~IO1
Routing:
- net GND: track 0.00 -> 106.5 mm
- net /~RST: track 0.00 -> 97.2 mm, vias 0 -> 5
- net /~IO1: track 0.00 -> 74.2 mm, vias 0 -> 1
- net +5V: track 0.00 -> 71.0 mm
- net /~CE: track 0.00 -> 61.9 mm, vias 0 -> 3
- net /A0: track 0.00 -> 56.0 mm, vias 0 -> 1
- net /~WE: track 0.00 -> 55.2 mm, vias 0 -> 1
- net /A15: track 0.00 -> 54.9 mm, vias 0 -> 1
- net /A14: track 0.00 -> 54.7 mm
- net /D2: track 0.00 -> 52.4 mm, vias 0 -> 2
- net /D3: track 0.00 -> 51.3 mm, vias 0 -> 2
- net /A3: track 0.00 -> 50.7 mm
- net /A1: track 0.00 -> 50.6 mm, vias 0 -> 1
- net /A13: track 0.00 -> 50.6 mm
- net /~ROMH: track 0.00 -> 50.4 mm
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