File: c64-umd/c64-umd.sch (KiCad schematic (older format))
At the start: 6 parts

Commit message: prelim sch done
Parts:
- removed C?: 10uF/10V, db-smt:0805, symbol C_0805
- added D101: BAT54A, db-smt:SOT23, symbol BAT54A
- added Q101: MMBT3904LT1G, SOT-23, symbol MMBT3904LT1G
- added R101, R102, R103: 10.0k, db-smt:0603, symbol R_0603
- gave numbers to parts that had none: 4
Connections:
- net labels added: +5V, A0, A1, A10, A11, A12, A13, A14, A15, A2, A3, A4, A5, A6, A7, A8, A9, D0, D1, D2, D3, D4, D5, D6, D7, GND, MISO, Phi2, SCK, ~CE, ~EXROM, ~GAME, ~ID, ~IO1, ~IO2, ~ROMH, ~ROML, ~RST, ~WE
- wire segments 0 -> 143
Other:
- note added: "ID = 0x02"
- moved on the sheet: C101, CON101, CON102A, CON102B, U101

Commit message: pcb outline and parts layout
Parts:
- removed Q101: MMBT3904LT1G, SOT-23, symbol MMBT3904LT1G
- added Q101: SMMBT3904LT1G, db-smt:SOT23, symbol SMMBT3904LT1G
Connections:
- wire segments 143 -> 126
Changed lines of the file:
@@
 $EndComp
 $Comp
-L GND #PWR104
+L GND #PWR01
 U 1 1 5ABBBFE9
 P 3500 6300
-F 0 "#PWR104" H 3500 6050 50  0001 C CNN
+F 0 "#PWR01" H 3500 6050 50  0001 C CNN
 F 1 "GND" H 3500 6150 50  0000 C CNN
 F 2 "" H 3500 6300 50  0001 C CNN
@@
 $EndComp
 $Comp
-L +5V #PWR102
+L +5V #PWR02
 U 1 1 5ABBC009
 P 2550 4800
-F 0 "#PWR102" H 2550 4650 50  0001 C CNN
+F 0 "#PWR02" H 2550 4650 50  0001 C CNN
 F 1 "+5V" H 2550 4940 50  0000 C CNN
 F 2 "" H 2550 4800 50  0001 C CNN
@@
 MISO
 $Comp
-L GND #PWR107
+L GND #PWR03
 U 1 1 5ABBC15D
 P 4850 5400
-F 0 "#PWR107" H 4850 5150 50  0001 C CNN
+F 0 "#PWR03" H 4850 5150 50  0001 C CNN
 F 1 "GND" H 4850 5250 50  0000 C CNN
 F 2 "" H 4850 5400 50  0001 C CNN
@@
 	4700 5300 4850 5300
 Wire Wire Line
-	4850 4900 4850 5300
-Wire Wire Line
-	4850 5300 4850 5400
-Wire Wire Line
-	4200 5300 4300 5300
-Wire Wire Line
-	4300 5300 4400 5300
+	4850 4900 4850 5400
+Wire Wire Line
+	4200 5300 4400 5300
 $Comp
 L R_0603 R102
@@
 $EndComp
 Wire Wire Line
-	3500 6000 3500 6250
-Wire Wire Line
-	3500 6250 3500 6300
-$Comp
-L MMBT3904LT1G Q101
-U 1 1 5ABBD2B0
-P 2450 6000
-F 0 "Q101" H 2650 6075 50  0000 L CNN
-F 1 "MMBT3904LT1G" H 2650 6000 50  0000 L CNN
-F 2 "SOT-23" H 2650 5925 50  0001 L CIN
-F 3 "" H 2450 6000 50  0000 L CNN
-	1    2450 6000
-	1    0    0    -1
-$EndComp
+	3500 6000 3500 6300
 $Comp
 L R_0603 R101
@@
 $EndComp
 Wire Wire Line
-	2550 4800 2550 4850
-Wire Wire Line
-	2550 4850 2550 4900
-Wire Wire Line
-	2550 4850 2700 4850
-Wire Wire Line
-	2700 4850 3750 4850
-Wire Wire Line
-	3750 4850 4300 4850
+	2550 4800 2550 4900
+Wire Wire Line
+	2550 4850 4300 4850
 Wire Wire Line
 	4300 4850 4300 5300
@@
 	3150 4950 3150 4900
 Wire Wire Line
-	3150 4900 3250 4900
-Wire Wire Line
-	3250 4900 3350 4900
-Wire Wire Line
-	3350 4900 3450 4900
-Wire Wire Line
-	3450 4900 3550 4900
-Wire Wire Line
-	3550 4900 3650 4900
-Wire Wire Line
-	3650 4900 3850 4900
-Wire Wire Line
-	3850 4900 4850 4900
+	3150 4900 4850 4900
 Connection ~ 4850 5300
 Wire Wire Line
@@
 Connection ~ 3850 4900
 Wire Wire Line
-	2550 5300 2550 5700
-Wire Wire Line
-	2550 5700 2550 5800
+	2550 5300 2550 5800
 Wire Wire Line
 	2550 6200 2550 6250
@@
 ID = 0x02
 $Comp
-L GND #PWR105
+L GND #PWR04
 U 1 1 5ABBDD30
 P 4150 4050
-F 0 "#PWR105" H 4150 3800 50  0001 C CNN
+F 0 "#PWR04" H 4150 3800 50  0001 C CNN
 F 1 "GND" H 4150 3900 50  0000 C CNN
 F 2 "" H 4150 4050 50  0001 C CNN
@@
 $EndComp
 $Comp
-L GND #PWR103
+L GND #PWR05
 U 1 1 5ABBDD53
 P 2950 4050
-F 0 "#PWR103" H 2950 3800 50  0001 C CNN
+F 0 "#PWR05" H 2950 3800 50  0001 C CNN
 F 1 "GND" H 2950 3900 50  0000 C CNN
 F 2 "" H 2950 4050 50  0001 C CNN
@@
 	4100 3950 4150 3950
 Wire Wire Line
-	4150 1850 4150 3950
-Wire Wire Line
-	4150 3950 4150 4050
-$Comp
-L +5V #PWR106
+	4150 1850 4150 4050
+$Comp
+L +5V #PWR06
 U 1 1 5ABBDDE2
 P 4650 3700
-F 0 "#PWR106" H 4650 3550 50  0001 C CNN
+F 0 "#PWR06" H 4650 3550 50  0001 C CNN
 F 1 "+5V" H 4650 3840 50  0000 C CNN
 F 2 "" H 4650 3700 50  0001 C CNN
@@
 $EndComp
 Wire Wire Line
-	4100 3750 4200 3750
-Wire Wire Line
-	4200 3750 4650 3750
+	4100 3750 4650 3750
 Wire Wire Line
 	4100 3850 4200 3850
@@
 MISO
 $Comp
-L GND #PWR109
+L GND #PWR07
 U 1 1 5ABBF6F2
 P 7950 5100
-F 0 "#PWR109" H 7950 4850 50  0001 C CNN
+F 0 "#PWR07" H 7950 4850 50  0001 C CNN
 F 1 "GND" H 7950 4950 50  0000 C CNN
 F 2 "" H 7950 5100 50  0001 C CNN
@@
 $EndComp
 Wire Wire Line
-	8000 5000 7950 5000
-Wire Wire Line
-	7950 1900 7950 2800
-Wire Wire Line
-	7950 2800 7950 5000
-Wire Wire Line
-	7950 5000 7950 5100
+	7950 5000 8000 5000
+Wire Wire Line
+	7950 1900 7950 5100
 Wire Wire Line
 	8000 2800 7950 2800
@@
 A13
 $Comp
-L GND #PWR108
+L GND #PWR08
 U 1 1 5ABC159E
 P 6400 5100
-F 0 "#PWR108" H 6400 4850 50  0001 C CNN
+F 0 "#PWR08" H 6400 4850 50  0001 C CNN
 F 1 "GND" H 6400 4950 50  0000 C CNN
 F 2 "" H 6400 5100 50  0001 C CNN
@@
 $EndComp
 Wire Wire Line
-	6450 5000 6400 5000
-Wire Wire Line
-	6400 5000 6400 5000
-Wire Wire Line
-	6400 5000 6400 5100
+	6400 5000 6450 5000
+Wire Wire Line
+	6400 1900 6400 5100
 Wire Wire Line
 	6450 2200 6050 2200
@@
 ~CE
 Wire Wire Line
-	2300 3950 2400 3950
-Wire Wire Line
-	2400 3950 3000 3950
+	2300 3950 3000 3950
 Text Label 1600 3875 0    60   ~ 0
 ~CE
@@
 $EndComp
 $Comp
-L +5V #PWR101
+L +5V #PWR09
 U 1 1 5ABC4213
 P 2400 3300
-F 0 "#PWR101" H 2400 3150 50  0001 C CNN
+F 0 "#PWR09" H 2400 3150 50  0001 C CNN
 F 1 "+5V" H 2400 3440 50  0000 C CNN
 F 2 "" H 2400 3300 50  0001 C CNN
@@
 $EndComp
 $Comp
-L +5V #PWR?
+L +5V #PWR010
 U 1 1 5ABC4F75
 P 5900 1850
-F 0 "#PWR?" H 5900 1700 50  0001 C CNN
+F 0 "#PWR010" H 5900 1700 50  0001 C CNN
 F 1 "+5V" H 5900 1990 50  0000 C CNN
 F 2 "" H 5900 1850 50  0001 C CNN
@@
 	6450 2000 5900 2000
 Wire Wire Line
-	5900 1850 5900 2000
-Wire Wire Line
-	5900 2000 5900 2800
+	5900 1850 5900 2800
 Wire Wire Line
 	5900 2800 6450 2800
@@
 Wire Wire Line
 	6450 1900 6400 1900
-Wire Wire Line
-	6400 1900 6400 5000
 Connection ~ 6400 5000
 $Bitmap
@@
 EndData
 $EndBitmap
+$Comp
+L SMMBT3904LT1G Q101
+U 1 1 5ABC372D
+P 2450 6000
+F 0 "Q101" H 2650 6075 50  0000 L CNN
+F 1 "SMMBT3904LT1G" H 2650 6000 50  0000 L CNN
+F 2 "db-smt:SOT23" H 2650 5925 50  0001 L CIN
+F 3 "http://www.onsemi.com/pub/Collateral/MMBT3904LT1-D.PDF" H 2475 6325 50  0001 L CNN
+F 4 "SMMBT3904LT1GOSCT-ND" H 3050 6400 60  0001 C CNN "Digikey"
+F 5 "TRANS NPN 40V 0.2A SOT23" H 3100 6500 60  0001 C CNN "Description"
+	1    2450 6000
+	1    0    0    -1
+$EndComp
+$Comp
+L +5V #PWR?
+U 1 1 5ABC5209
+P 5900 4850
+F 0 "#PWR?" H 5900 4700 50  0001 C CNN
+F 1 "+5V" H 5900 4990 50  0000 C CNN
+F 2 "" H 5900 4850 50  0001 C CNN
+F 3 "" H 5900 4850 50  0001 C CNN
+	1    5900 4850
+	1    0    0    -1
+$EndComp
+Wire Wire Line
+	5900 4850 5900 4900
+Wire Wire Line
+	5900 4900 6450 4900
+$Comp
+L +5V #PWR?
+U 1 1 5ABC53B2
+P 7450 4850
+F 0 "#PWR?" H 7450 4700 50  0001 C CNN
+F 1 "+5V" H 7450 4990 50  0000 C CNN
+F 2 "" H 7450 4850 50  0001 C CNN
+F 3 "" H 7450 4850 50  0001 C CNN
+	1    7450 4850
+	1    0    0    -1
+$EndComp
+Wire Wire Line
+	7450 4850 7450 4900
+Wire Wire Line
+	7450 4900 8000 4900
 $EndSCHEMATC

Commit message: prelim routing complete, review before 0.1 release
Connections:
- wire segments 126 -> 124
Changed lines of the file:
@@
 Wire Wire Line
 	7950 1900 7950 5100
-Wire Wire Line
-	8000 2800 7950 2800
 Connection ~ 7950 5000
 Wire Wire Line
@@
 Wire Wire Line
 	6450 2200 6050 2200
-Text Label 6050 2200 0    60   ~ 0
+Text Label 6050 2500 0    60   ~ 0
 ~ROMH
 Wire Wire Line
@@
 Wire Wire Line
 	8000 2200 7600 2200
-Text Label 7600 2200 0    60   ~ 0
+Text Label 7600 2300 0    60   ~ 0
 ~IO2
 Wire Wire Line
@@
 Wire Wire Line
 	6450 2400 6050 2400
-Text Label 6050 2400 0    60   ~ 0
+Text Label 6050 2300 0    60   ~ 0
 ~GAME
 Wire Wire Line
 	6450 2300 6050 2300
-Text Label 6050 2300 0    60   ~ 0
+Text Label 6050 2200 0    60   ~ 0
 ~EXROM
 Wire Wire Line
@@
 Wire Wire Line
 	6450 2600 6050 2600
-Text Label 6050 2600 0    60   ~ 0
+Text Label 7600 2200 0    60   ~ 0
 ~ROML
 Wire Wire Line
@@
 Wire Wire Line
 	6450 2500 6050 2500
-Text Label 6050 2500 0    60   ~ 0
+Text Label 6050 2600 0    60   ~ 0
 ~IO1
 Wire Wire Line
 	8000 2300 7600 2300
-Text Label 7600 2300 0    60   ~ 0
+Text Label 6050 2400 0    60   ~ 0
 Phi2
 Wire Wire Line
@@
 	6450 2000 5900 2000
 Wire Wire Line
-	5900 1850 5900 2800
-Wire Wire Line
-	5900 2800 6450 2800
-Connection ~ 5900 2000
-Wire Wire Line
 	8000 1900 7950 1900
-Connection ~ 7950 2800
 Wire Wire Line
 	6450 1900 6400 1900
@@
 $EndComp
 $Comp
-L +5V #PWR?
+L +5V #PWR011
 U 1 1 5ABC5209
 P 5900 4850
-F 0 "#PWR?" H 5900 4700 50  0001 C CNN
+F 0 "#PWR011" H 5900 4700 50  0001 C CNN
 F 1 "+5V" H 5900 4990 50  0000 C CNN
 F 2 "" H 5900 4850 50  0001 C CNN
@@
 	5900 4900 6450 4900
 $Comp
-L +5V #PWR?
+L +5V #PWR012
 U 1 1 5ABC53B2
 P 7450 4850
-F 0 "#PWR?" H 7450 4700 50  0001 C CNN
+F 0 "#PWR012" H 7450 4700 50  0001 C CNN
 F 1 "+5V" H 7450 4990 50  0000 C CNN
 F 2 "" H 7450 4850 50  0001 C CNN
@@
 Wire Wire Line
 	7450 4900 8000 4900
+Wire Wire Line
+	5900 2000 5900 1850
 $EndSCHEMATC
